Commit message: Simplify kitten face and smooth cosmetic limb surfaces

File: concepts/cat-layout-v4/robot.urdf (robot description, URDF)
Before this commit: robot kitten_v4_layout, 20 links, 19 joints
Links:
- link front_L_elbow: geometry collision box size=0.022 0.022 0.13; collision sphere radius=0.035
- link front_R_elbow: geometry collision box size=0.022 0.022 0.13; collision sphere radius=0.035
- link neck_pitch: geometry collision cylinder length=0.03 radius=0.02; visual cylinder length=0.004 radius=0.0144
